Commit message: FEAT: added Kinect RGBD camera for SLAM

File: P4-MapMyWorld/catkin_ws/src/my_robot/urdf/my_robot.xacro (robot description, xacro)
@@ -166,4 +166,12 @@
         <axis xyz="0 1 0"/>
    </joint>
+  <!-- Kinect Camera for Project 4-->
+  <joint name="camera_optical_joint" type="fixed">
+    <origin xyz="0 0 0" rpy="-1.5707 0 -1.5707"/>
+    <parent link="camera_link"/>
+    <child link="camera_link_optical"/>
+  </joint>
+  <link name="camera_link_optical">
+  </link>
  <!-- Lidar: Hokuyo -->
   <link name="hokuyo">

Commit message: fixed: camera link name

File: P4-MapMyWorld/catkin_ws/src/my_robot/urdf/my_robot.xacro (robot description, xacro)
@@ -169,5 +169,5 @@
   <joint name="camera_optical_joint" type="fixed">
     <origin xyz="0 0 0" rpy="-1.5707 0 -1.5707"/>
-    <parent link="camera_link"/>
+    <parent link="camera"/>
     <child link="camera_link_optical"/>
   </joint>
